File: hardware/04_power_supply.kicad_sch (KiCad schematic)
At the start: 12 parts, among them U4 LMR16006XDDCR (Tokmas)

Commit message: 知识库：pgrep 自匹配僵尸等待循环教训
Co-Authored-By: Claude Opus 5.5 <noreply@anthropic.com>
Claude-Session: https://claude.ai/code/session_018LcBBXJnjJ1MVmds7Fkezv
Parts:
- added C45: 100nF 100V, jlc:C0805, symbol jlc:CL21B104KCFNNNE
- R42: value 10Ω 1% 1206 -> 56Ω 5% 熔断 1206; symbol jlc:1206W4F100JT5E -> jlc:FCR1206J56RP055W; LCSC C17903 -> C153337
Connections:
- net GND: now also C45.1
- net VIN_F: now also C45.2
Other:
- note added: "R42 56Ω 熔断电阻与 C40 构成输入 RC：限上电浪涌与短路电流，VIN_F 短路时受控开路；C45 100nF/100V 贴 VIN（Tokmas 手册 p14）"
- note removed: "R42 10Ω 与 C40 构成输入 RC：限上电浪涌与短路电流，替代已删的 D6；L1 下方全层禁铜（规则 2d）"
- moved on the sheet: C42, C44
Changed lines of the file:
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@@
 		(title "辅助电源")
 		(date "2026-09-26")
-		(rev "v0.3-draw-r4")
+		(rev "v0.3-draw-r5")
 		(company "MP2645A-BMS")
 		(comment 1 "8S LiFePO4 200A BMS · MPS MP2797 + 开关电容均衡")
@@
 		)
 	)
-	(text "R42 10Ω 与 C40 构成输入 RC：限上电浪涌与短路电流，替代已删的 D6；L1 下方全层禁铜（规则 2d）"
+	(text "R42 56Ω 熔断电阻与 C40 构成输入 RC：限上电浪涌与短路电流，VIN_F 短路时受控开路；C45 100nF/100V 贴 VIN（Tokmas 手册 p14）"
 		(exclude_from_sim no)
 		(at 40.64 38.10 0)
@@
 	(global_label "GND"
 		(shape input)
+		(at 266.70 121.92 0)
+		(effects
+			(font
+				(size 1.27 1.27)
+			)
+			(justify left)
+		)
+	)
+	(global_label "GND"
+		(shape input)
 		(at 233.68 96.52 0)
 		(effects
@@
 	(wire
 		(pts
-			(xy 215.90 114.30)
+			(xy 241.30 104.14)
+			(xy 266.70 104.14)
+		)
+		(stroke
+			(width 0)
+			(type default)
+		)
+	)
+	(wire
+		(pts
+			(xy 215.90 111.76)
 			(xy 215.90 121.92)
 		)
@@
 	(wire
 		(pts
+			(xy 266.70 114.30)
+			(xy 266.70 121.92)
+		)
+		(stroke
+			(width 0)
+			(type default)
+		)
+	)
+	(wire
+		(pts
 			(xy 223.52 80.01)
 			(xy 223.52 71.12)
@@
 	)
 	(junction (at 304.80 71.12) (diameter 0) (color 0 0 0 0))
+	(junction (at 215.90 104.14) (diameter 0) (color 0 0 0 0))
+	(junction (at 241.30 104.14) (diameter 0) (color 0 0 0 0))
+	(junction (at 289.56 71.12) (diameter 0) (color 0 0 0 0))
 	(no_connect (at 195.58 106.68))
 	(symbol
@@
 	)
 	(symbol
-		(lib_id "jlc:1206W4F100JT5E")
+		(lib_id "jlc:FCR1206J56RP055W")
 		(at 114.30 71.12 0)
 		(unit 1)
@@
 			)
 		)
-		(property "Value" "10Ω 1% 1206"
+		(property "Value" "56Ω 5% 熔断 1206"
 			(at 114.30 73.66 0)
 			(effects
@@
 			)
 		)
-		(property "Datasheet" "https://lcsc.com/product-detail/Chip-Resistor-Surface-Mount-UniOhm_10R-10R0-1_C17903.html"
+		(property "Datasheet" "https://lcsc.com/product-detail/Fusible-Chip-Resistor_Ever-Ohms-Tech-FCR1206J56RP055W_C153337.html"
 			(at 114.30 78.74 0)
 			(effects
@@
 			)
 		)
-		(property "LCSC" "C17903"
+		(property "LCSC" "C153337"
 			(at 114.30 78.74 0)
 			(effects
@@
 			)
 		)
-		(property "Datasheet" "https://lcsc.com/product-detail/Switching-Controllers_TI_LMR16006XDDCR_LMR16006XDDCR_C87080.html"
+		(property "Datasheet" "https://www.lcsc.com/datasheet/C54823941.pdf"
 			(at 185.42 111.76 0)
 			(effects
@@
 	)
 	(symbol
-		(lib_id "jlc:CL31B105KCHNNNE")
-		(at 215.90 109.22 90)
+		(lib_id "jlc:CL21B104KCFNNNE")
+		(at 215.90 107.95 90)
 		(unit 1)
 		(exclude_from_sim no)
@@
 		(on_board yes)
 		(dnp no)
-		(property "Reference" "C42"
-			(at 220.98 106.68 270)
-			(effects
-				(font
-					(size 1.27 1.27)
-				)
-				(justify left)
-			)
-		)
-		(property "Value" "1µF 100V"
-			(at 220.98 111.76 270)
-			(effects
-				(font
-					(size 1.27 1.27)
-				)
-				(justify left)
-			)
-		)
-		(property "Footprint" "jlc:C1206"
-			(at 215.90 116.84 0)
-			(effects
-				(font
-					(size 1.27 1.27)
-				)
-				(justify left)
-				hide
-			)
-		)
-		(property "Datasheet" "https://lcsc.com/product-detail/Multilayer-Ceramic-Capacitors-MLCC-SMD-SMT_SAMSUNG_CL31B105KCHNNNE_1uF-105-10-100V_C13832.html"
-			(at 215.90 116.84 0)
-			(effects
-				(font
-					(size 1.27 1.27)
-				)
-				(justify left)
-				hide
-			)
-		)
-		(property "LCSC" "C13832"
-			(at 215.90 116.84 0)
+		(property "Reference" "C45"
+			(at 220.98 105.41 270)
+			(effects
+				(font
+					(size 1.27 1.27)
+				)
+				(justify left)
+			)
+		)
+		(property "Value" "100nF 100V"
+			(at 220.98 110.49 270)
+			(effects
+				(font
+					(size 1.27 1.27)
+				)
+				(justify left)
+			)
+		)
+		(property "Footprint" "jlc:C0805"
+			(at 215.90 115.57 0)
+			(effects
+				(font
+					(size 1.27 1.27)
+				)
+				(justify left)
+				hide
+			)
+		)
+		(property "Datasheet" "https://lcsc.com/product-detail/Multilayer-Ceramic-Capacitors-MLCC-SMD-SMT_SAMSUNG_CL21B104KCFNNNE_100nF-104-10-100V_C28233.html"
+			(at 215.90 115.57 0)
+			(effects
+				(font
+					(size 1.27 1.27)
+				)
+				(justify left)
+				hide
+			)
+		)
+		(property "LCSC" "C28233"
+			(at 215.90 115.57 0)
 			(effects
 				(font
@@
 			(project "mp2645a-bms"
 				(path "/632f74a5-cd8f-58d8-9ac1-1bfbb611d555/c20e45f9-c9d2-50e9-b477-f2356556af13"
-					(reference "C42")
+					(reference "C45")
 					(unit 1)
 				)
@@
 		(on_board yes)
 		(dnp no)
-		(property "Reference" "C44"
+		(property "Reference" "C42"
 			(at 246.38 106.68 270)
 			(effects
@@
 			(effects
 				(font
+					(size 1.27 1.27)
+				)
+				(justify left)
+				hide
+			)
+		)
+		(pin "1")
+		(pin "2")
+		(instances
+			(project "mp2645a-bms"
+				(path "/632f74a5-cd8f-58d8-9ac1-1bfbb611d555/c20e45f9-c9d2-50e9-b477-f2356556af13"
+					(reference "C42")
+					(unit 1)
+				)
+			)
+		)
+	)
+	(symbol
+		(lib_id "jlc:CL31B105KCHNNNE")
+		(at 266.70 109.22 90)
+		(unit 1)
+		(exclude_from_sim no)
+		(in_bom yes)
+		(on_board yes)
+		(dnp no)
+		(property "Reference" "C44"
+			(at 271.78 106.68 270)
+			(effects
+				(font
+					(size 1.27 1.27)
+				)
+				(justify left)
+			)
+		)
+		(property "Value" "1µF 100V"
+			(at 271.78 111.76 270)
+			(effects
+				(font
+					(size 1.27 1.27)
+				)
+				(justify left)
+			)
+		)
+		(property "Footprint" "jlc:C1206"
+			(at 266.70 116.84 0)
+			(effects
+				(font
+					(size 1.27 1.27)
+				)
+				(justify left)
+				hide
+			)
+		)
+		(property "Datasheet" "https://lcsc.com/product-detail/Multilayer-Ceramic-Capacitors-MLCC-SMD-SMT_SAMSUNG_CL31B105KCHNNNE_1uF-105-10-100V_C13832.html"
+			(at 266.70 116.84 0)
+			(effects
+				(font
+					(size 1.27 1.27)
+				)
+				(justify left)
+				hide
+			)
+		)
+		(property "LCSC" "C13832"
+			(at 266.70 116.84 0)
+			(effects
+				(font

Commit message: 04：C42/C44 按用户 14:46 决定改 C282823（脚本清单替换）；换符号后版面自检失败 → 第 6 轮任务书
Co-Authored-By: Claude Opus 5.5 <noreply@anthropic.com>
Claude-Session: https://claude.ai/code/session_018LcBBXJnjJ1MVmds7Fkezv
Parts:
- C42, C44: symbol jlc:CL31B105KCHNNNE -> jlc:TCC1206X7R105K101HT; LCSC C13832 -> C282823
Changed lines of the file:
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@@
 		(pts
 			(xy 215.90 104.14)
-			(xy 241.30 104.14)
-		)
-		(stroke
-			(width 0)
-			(type default)
-		)
-	)
-	(wire
-		(pts
-			(xy 241.30 104.14)
-			(xy 266.70 104.14)
+			(xy 236.22 109.22)
+		)
+		(stroke
+			(width 0)
+			(type default)
+		)
+	)
+	(wire
+		(pts
+			(xy 236.22 109.22)
+			(xy 261.62 109.22)
 		)
 		(stroke
@@
 	(wire
 		(pts
-			(xy 241.30 114.30)
+			(xy 246.38 109.22)
 			(xy 241.30 121.92)
 		)
@@
 	(wire
 		(pts
-			(xy 266.70 114.30)
+			(xy 271.78 109.22)
 			(xy 266.70 121.92)
 		)
@@
 	)
 	(symbol
-		(lib_id "jlc:CL31B105KCHNNNE")
+		(lib_id "jlc:TCC1206X7R105K101HT")
 		(at 241.30 109.22 90)
 		(unit 1)
@@
 			)
 		)
-		(property "Datasheet" "https://lcsc.com/product-detail/Multilayer-Ceramic-Capacitors-MLCC-SMD-SMT_SAMSUNG_CL31B105KCHNNNE_1uF-105-10-100V_C13832.html"
+		(property "Datasheet" "https://lcsc.com/product-detail/High-Voltage-Capacitors_CCTC-TCC1206X7R105K101HT_C282823.html"
 			(at 241.30 116.84 0)
 			(effects
@@
 			)
 		)
-		(property "LCSC" "C13832"
+		(property "LCSC" "C282823"
 			(at 241.30 116.84 0)
 			(effects
@@
 	)
 	(symbol
-		(lib_id "jlc:CL31B105KCHNNNE")
+		(lib_id "jlc:TCC1206X7R105K101HT")
 		(at 266.70 109.22 90)
 		(unit 1)
@@
 			)
 		)
-		(property "Datasheet" "https://lcsc.com/product-detail/Multilayer-Ceramic-Capacitors-MLCC-SMD-SMT_SAMSUNG_CL31B105KCHNNNE_1uF-105-10-100V_C13832.html"
+		(property "Datasheet" "https://lcsc.com/product-detail/High-Voltage-Capacitors_CCTC-TCC1206X7R105K101HT_C282823.html"
 			(at 266.70 116.84 0)
 			(effects
@@
 			)
 		)
-		(property "LCSC" "C13832"
+		(property "LCSC" "C282823"
 			(at 266.70 116.84 0)
 			(effects
