File: hardware/02_afe.kicad_sch (KiCad schematic)
At the start: 0 parts

Commit message: 02 页分段 A（deepseek-flash）：U1 48 脚、电源、高边驱动，自检 9 项通过；C219B→C226（KiCad 位号不能以字母结尾）
Co-Authored-By: Claude Opus 5.5 <noreply@anthropic.com>
Claude-Session: https://claude.ai/code/session_018LcBBXJnjJ1MVmds7Fkezv
Parts:
- added C212: 470nF 100V, jlc:C0805, symbol jlc:TCC0805X7R474K101FT
- added C213: 1µF 100V, jlc:C1206, symbol jlc:TCC1206X7R105K101HT
- added C214: 10µF 10V, jlc:C0603, symbol jlc:CL10A106KP8NNNC
- added C215, C216, C217: 1µF 25V, jlc:C0402, symbol jlc:CL05A105KA5NQNC
- added C218: 10nF 50V, jlc:C0402, symbol jlc:CL05B103KB5NNNC
- added C219, C220: 100nF 100V, jlc:C0805, symbol jlc:CL21B104KCFNNNE
- added C221: 10nF 100V, jlc:C0603, symbol jlc:TCC0603X7R103K101CT
- added C226: 100nF 100V DNP, jlc:C0805, symbol jlc:CL21B104KCFNNNE
- added Q201: MMBT5551, jlc:SOT-23-3_L2.9-W1.3-P1.90-LS2.4-BR, symbol jlc:MMBT5551_C2145
- added R212: 20Ω 1%, jlc:R0603, symbol jlc:0603WAF200JT5E
- added R213: 510Ω 1%, jlc:R0603, symbol jlc:0603WAF5100T5E
- added R214, R215: 100Ω 1%, jlc:R0402, symbol jlc:0402WGF1000TCE
- added U1: MP2797DFP-0000-T, jlc:LQFP-48_L7.0-W7.0-P0.50-LS9.0-BL_1, symbol jlc:MP2797DFP-0000-T
Connections:
- new net AFE_3V3: C215.2, U1.26 (3V3)
- new net AFE_ALERT: U1.28 (XALERT)
- new net AFE_VDD: C216.2, U1.27 (VDD)
- new net AFE_VREF: C217.2, U1.22 (VREF)
- new net AFE_WAKE: U1.30 (NSHDN)
- new net BAT+: R212.1, R213.1
- new net CHG_G: U1.44 (CHG)
- new net DSG_G: U1.39 (DSG)
- new net FET_MID: R214.1
- new net GND: C212.1, C213.1, C214.1, C215.1, C216.1, C217.1, C218.1, C220.1, C221.1, U1.23 (AGND)
- new net I2C_SCL: U1.31 (SCL/SCK)
- new net I2C_SDA: U1.32 (SDA/SDI)
- new net NTCB: C218.2, U1.21 (NTCB)
- new net NTC_CELL1: U1.20 (NTC1)
- new net NTC_CELL2: U1.19 (NTC2)
- new net NTC_FET: U1.18 (NTC3)
- new net NTC_SHUNT: U1.17 (NTC4)
- new net PACK+: R215.1
- new net PACKP: C221.2, R215.2, U1.38 (PACKP)
- new net REGCTRL: Q201.1 (B), U1.24 (REGCTRL)
- new net REGIN: C214.2, Q201.2 (E), U1.25 (REGIN)
- new net REG_C: C213.2, Q201.3 (C), R213.2
- new net SRN_F: U1.16 (SRN)
- new net SRP_F: U1.15 (SRP)
- new net VC0: U1.14 (C0)
- new net VC1: U1.13 (C1)
- new net VC2: U1.12 (C2)
- new net VC3: U1.11 (C3)
- new net VC4: U1.10 (C4)
- new net VC5: U1.9 (C5)
- new net VC6: U1.8 (C6)
- new net VC7: U1.7 (C7)
- new net VC8: U1.1 (C13), U1.2 (C12), U1.3 (C11), U1.4 (C10), U1.46 (C16), U1.47 (C15), U1.48 (C14), U1.5 (C9), U1.6 (C8)
- new net VCP: C219.2, C226.2, U1.42 (VCP)
- new net VMID: C219.1, C220.2, C226.1, R214.2, U1.43 (VMID)
- new net VTOP: C212.2, R212.2, U1.45 (VTOP)
- no-connect marks 0 -> 8
Other:
- note added: "02 AFE：MP2797 采集与保护（8S，C9–C16 并到 C8；WDT 悬空；xALERT 高有效 100k 下拉）"
- note added: "AFE_3V3 只接 C215，不与板上 +3V3 相连；NTC 四路上拉（R216–R219）都接 NTCB，不接任何 3V3。"
- note added: "C9–C16（脚 5,4,3,2,1,48,47,46）用一条竖线并在 C8（脚 6）的 VC8 上，不串电阻、不加电容（Table 23「directly connect」）。"
- note added: "U1 = MP2797DFP-0000-T（C18198873，TQFP-48）。本页 U1 全部引脚以「短线 + 标签」引出；未用脚放 NC 标志（29 WDT / 33 SDO / 34–37 GPIO / 40 N/C / 41 SBYDSG）。"
- note added: "U1.25 REGIN ← Q201(MMBT5551) 发射极；Q201 基极 = REGCTRL，集电极 = REG_C（C213 1µF/100V、R213 510Ω 到 BAT+）；C214 10µF/10V 贴 U1.25。"
- note added: "U1.38 PACKP ← R215 100Ω ← PACK+，C221 10nF/100V 到 GND（Table 18「不得增减」）。"
- note added: "U1.42 VCP ↔ VMID 跨接 C219 100nF/100V；C226 为扩展焊盘（DNP，样板实测 VCP 跌落后再定）。U1.44 CHG、U1.39 DSG 本页不串件，R_DRV/DZ/PNP 快关在 01 页。"
- note added: "U1.43 VMID ← R214 100Ω ← FET_MID，C220 100nF/100V 到 GND。"
- note added: "U1.45 VTOP ← R212 20Ω ← BAT+；C212 470nF/100V 在 VTOP 对 GND。"
- note added: "§6 高边驱动（CHG/DSG/VCP/VMID/PACKP）"
- note added: "§9 电源：BAT+ 供电（U-1）"
- note added: "分段 A 已画：U1 + §9 电源 + §6 高边驱动。J5/电芯采样 RC/NTC/通讯见分段 B、C。"
- note removed: "MP2797 采集与保护"
- note removed: "· +3V3"
- note removed: "· AFE_ALERT"
- note removed: "· AFE_WAKE"
- note removed: "· CELL0..CELL8"
- note removed: "· CHG_G"
- note removed: "· DSG_G"
- note removed: "· FET_MID"
- note removed: "· GND"
- note removed: "· I2C_SCL"
- note removed: "· I2C_SDA"
- note removed: "· NTC_CELL1"
- note removed: "· NTC_CELL2"
- note removed: "· NTC_FET"
- note removed: "· NTC_SHUNT"
- note removed: "· PACK+"
- note removed: "· SRN"
- note removed: "· SRP"
- note removed: "内容：电芯采样 RC / 电流采样滤波 / 4 路 NTC / 高边驱动输出 / 通讯与中断 / 被动均衡"
- note removed: "接口网络（跨页用全局标签，名称以本清单为准）："
- note removed: "状态：待画。详细设计见 docs/03-详细设计.md；按 pcb-workflow 规则 00/00c/00d 执行。"

Commit message: 02 页分段 B（电芯采样 RC、电流采样、J5；自检 9 项 140 脚通过）；分段 C 任务书
Co-Authored-By: Claude Opus 5.5 <noreply@anthropic.com>
Claude-Session: https://claude.ai/code/session_018LcBBXJnjJ1MVmds7Fkezv
Parts:
- added C201, C202, C203, C204, C205, C206, C207, C208: 100nF 50V, jlc:C0402, symbol jlc:CL05B104KB54PNC
- added C209, C210, C211: 100nF 50V, jlc:C0402, symbol jlc:CL05B104KO5NNNC
- added D201: BZT52C3V3, jlc:SOD-123_L2.8-W1.8-LS3.7-RD, symbol jlc:BZT52C3V3_C353528
- added J5: XH-13A 13P, jlc:CONN-TH_13P-P2.50_XH-13A, symbol jlc:XH-13A
- added R201, R202, R203, R204, R205, R206, R207, R208, R209: 33Ω 1%, jlc:R0805, symbol jlc:0805W8F330JT5E
- added R210, R211: 100Ω 1%, jlc:R0402, symbol jlc:0402WGF1000TCE
Connections:
- net GND: now also C210.1, C211.1, D201.2 (A), J5.2, J5.4
- net NTC_CELL1: now also J5.1
- net NTC_CELL2: now also J5.3
- net SRN_F: now also C209.2, C211.2, R211.2
- net SRP_F: now also C209.1, C210.2, R210.2
- net VC0: now also C201.1, D201.1 (C), R201.2
- net VC1: now also C201.2, C202.1, R202.2
- net VC2: now also C202.2, C203.1, R203.2
- net VC3: now also C203.2, C204.1, R204.2
- net VC4: now also C204.2, C205.1, R205.2
- net VC5: now also C205.2, C206.1, R206.2
- net VC6: now also C206.2, C207.1, R207.2
- net VC7: now also C207.2, C208.1, R208.2
- net VC8: now also C208.2, R209.2
- new net CELL0: J5.5, R201.1
- new net CELL1: J5.6, R202.1
- new net CELL2: J5.7, R203.1
- new net CELL3: J5.8, R204.1
- new net CELL4: J5.9, R205.1
- new net CELL5: J5.10, R206.1
- new net CELL6: J5.11, R207.1
- new net CELL7: J5.12, R208.1
- new net CELL8: J5.13, R209.1
- new net SRN: R211.1
- new net SRP: R210.1
Other:
- note added: "1 NTC_CELL1 / 2 GND / 3 NTC_CELL2 / 4 GND"
- note added: "5–13 = CELL0…CELL8。"
- note added: "C201–C208 100nF/50V 跨相邻两个 VC（8 只，不接地）；C0 只挂 D201 稳压（阴极→VC0、阳极→GND）。"
- note added: "C209 100nF 跨 SRP_F↔SRN_F（差模）；C210/C211 各 100nF 到 GND（共模）。"
- note added: "C40669 XH 2.50mm 13P 立式；"
- note added: "J5.5–13 CELL0–CELL8 → R201–R209 33Ω 1% → VC0–VC8 → U1.14/13/12/11/10/9/8/7/6。"
- note added: "NTC 放低压端（紧贴 CELL0–CELL8，"
- note added: "SRP/SRN 取自分流器电池侧（01 页），经 R210/R211 100Ω → SRP_F/SRN_F → U1.15/U1.16。"
- note added: "§10 J5 采样端子"
- note added: "§4 电芯采样 RC（9 串）"
- note added: "§5 电流采样（SRP/SRN 开尔文）"
- note added: "分段 A+B 已画：U1 + §9 电源 + §6 驱动 + §4 电芯 RC + §5 采样 + §10 J5；NTC/通讯见分段 C。"
- note added: "均衡电流走串阻：33Ω 时典型 39mA、最坏 45mA，0805 耗散余量 1.5 倍；本页不出现任何 BAL* 标签。"
- note added: "线束短路不会把 29V 灌进 NTC 脚）。"
- note removed: "分段 A 已画：U1 + §9 电源 + §6 高边驱动。J5/电芯采样 RC/NTC/通讯见分段 B、C。"
